Commit message: reorganized project, finished xacro file

File: src/differential_drive_description/model/robot.xacro (robot description, xacro)
@@ -2,5 +2,4 @@
 <robot xmlns:xacro="http://www.ros.org/wiki/xacro" name="differential_drive_robot">
 <!--- Constants -->
-<xacro:property name="pi" value="3.14159265" />
 <!--- Body dimensions -->
 <xacro:property name="a" value="1" />
@@ -55,5 +54,5 @@
     </inertial>
 </xacro:macro>
-<xacro:include filename="$(find differential-drive-ws)/model/robot.gazebo" />
+<!--- <xacro:include filename="$(find differential_drive_description)/model/robot.gazebo" /> -->
 <link name="base_footprint"> </link>
 <joint name="body_link_joint" type="fixed">
@@ -64,5 +63,5 @@
     <visual>
         <geometry>
-            <box size="${a} ${b} ${c}"/>
+            <box size="${a} ${c} ${b}"/>
         </geometry>
         <origin rpy="0 0 0" xyz="0 0 ${s1}" />
@@ -70,5 +69,5 @@
     <collision>
         <geometry>
-            <box size="${a} ${b} ${c}"/>
+            <box size="${a} ${c} ${b}"/>
         </geometry>
         <origin rpy="0 0 0" xyz="0 0 ${s1}" />
@@ -76,3 +75,69 @@
     <xacro:inertia_body />
 </link>
+<joint name="wheel1_joint" type="continuous">
+    <parent link="body_link"/>
+    <child link="wheel1_link"/>
+    <origin xyz="${-s2} ${-s4} ${r}" rpy="0 0 0"/>
+    <axis xyz="0 1 0"/>
+    <limit effort="50000" velocity="10"/>
+    <dynamics damping="1.0" friction="1.0"/>
+</joint>
+<link name="wheel1_link">
+    <visual>
+        <origin rpy="1.570795 0 0" xyz="0 0 0"/>
+        <geometry>
+            <cylinder radius="${r}" length="${d}"/>
+        </geometry>
+    </visual>
+    <collision>
+        <origin rpy="1.570795 0 0" xyz="0 0 0"/>
+        <geometry>
+            <cylinder radius="${r}" length="${d}"/>
+        </geometry>
+    </collision>
+    <xacro:inertia_wheel/>
+</link>
+<joint name="wheel2_joint" type="continuous">
+    <parent link="body_link"/>
+    <child link="wheel2_link"/>
+    <origin xyz="${-s2} ${s4} ${r}" rpy="0 0 0"/>
+    <axis xyz="0 1 0"/>
+    <limit effort="50000" velocity="10"/>
+    <dynamics damping="1.0" friction="1.0"/>
+</joint>
+<link name="wheel2_link">
+    <visual>
+        <origin rpy="1.570795 0 0" xyz="0 0 0"/>
+        <geometry>
+            <cylinder radius="${r}" length="${d}"/>
+        </geometry>
+    </visual>
+    <collision>
+        <origin rpy="1.570795 0 0" xyz="0 0 0"/>
+        <geometry>
+            <cylinder radius="${r}" length="${d}"/>
+        </geometry>
+    </collision>
+    <xacro:inertia_wheel/>
+</link>
+<joint name="caster_joint" type="fixed">
+    <parent link="body_link"/>
+    <child link="caster_link"/>
+    <origin xyz="${s3} 0 ${r}" rpy="0 0 0"/>
+</joint>
+<link name="caster_link">
+    <visual>
+        <origin xyz="0 0 0" rpy="0 0 0"/>
+        <geometry>
+            <sphere radius="${r}"/>
+        </geometry>
+    </visual>
+    <collision>
+        <origin xyz="0 0 0" rpy="0 0 0"/>
+        <geometry>
+            <sphere radius="${r}"/>
+        </geometry>
+    </collision>
+    <xacro:inertia_caster/>
+</link>
 </robot>

Commit message: added a gazebo world and a lidar

File: src/differential_drive_description/model/robot.xacro (robot description, xacro)
@@ -3,10 +3,10 @@
 <!-- Constants -->
 <!-- Body dimensions -->
-<xacro:property name="a" value="1" />
-<xacro:property name="b" value="0.3" />
-<xacro:property name="c" value="0.6" />
+<xacro:property name="a" value="0.5" />
+<xacro:property name="b" value="0.15" />
+<xacro:property name="c" value="0.3" />
 <!-- Wheel and castor dimensions -->
-<xacro:property name="r" value="0.15" />
-<xacro:property name="d" value="0.1" />
+<xacro:property name="r" value="0.07" />
+<xacro:property name="d" value="0.05" />
 <xacro:property name="s1" value="${b/2+r}" />
 <xacro:property name="s2" value="${2*r}" />
@@ -141,3 +141,28 @@
     <xacro:inertia_caster/>
 </link>
+<joint name="lidar_joint" type="fixed">
+        <origin xyz="0 0 ${b+r}" rpy="0 0 0"/>
+        <parent link="body_link"/>
+        <child link="lidar_link"/>
+        <axis xyz="0 1 0" rpy="0 0 0"/>
+</joint>
+<link name="lidar_link">
+    <visual>
+        <origin xyz="0 0 0.025" rpy="0 0 0"/>
+        <geometry>
+            <cylinder radius="0.05" length="0.05"/>
+        </geometry>
+    </visual>
+    <geometry>
+        <origin xyz="0 0 0.025" rpy="0 0 0"/>
+        <geometry>
+            <cylinder radius="0.05" length="0.05"/>
+        </geometry>
+    </geometry>
+    <inertial>
+        <mass value="0.5e-6"/>
+        <origin xyz="0 0 0" rpy="0 0 0"/>
+        <inertia ixx="0.5e-6" ixy="0.0" ixz="0.0" iyy="0.5e-6" iyz="0.0" izz="0.5e-6"/>
+    </inertial>
+</link>
 </robot>
