Commit message: fixed material issue

File: src/mobile_robot/model/robot.xacro (robot description, xacro)
@@ -1,5 +1,11 @@
 <?xml version="1.0"?>
 <robot xmlns:xacro="http://www.ros.org/wiki/xacro" name="differential_drive_robot">
-<!-- Constants -->
+<!-- Materials -->
+<material name="black">
+  <color rgba="0.01 0.01 0.01 1"/>
+</material>
+<material name="green">
+  <color rgba="0.1 0.9 0.2 1"/>
+</material>
 <!-- Body dimensions -->
 <xacro:property name="a" value="0.5" />
@@ -66,4 +72,5 @@
         </geometry>
         <origin rpy="0 0 0" xyz="0 0 ${s1}" />
+        <material name="black"/>
     </visual>
     <collision>
@@ -89,4 +96,5 @@
             <cylinder radius="${r}" length="${d}"/>
         </geometry>
+        <material name="green"/>
     </visual>
     <collision>
@@ -112,4 +120,5 @@
             <cylinder radius="${r}" length="${d}"/>
         </geometry>
+        <material name="green"/>
     </visual>
     <collision>
@@ -132,4 +141,5 @@
             <sphere radius="${r}"/>
         </geometry>
+        <material name="green"/>
     </visual>
     <collision>
@@ -153,4 +163,5 @@
             <cylinder radius="0.05" length="0.05"/>
         </geometry>
+        <material name="black"/>
     </visual>
     <geometry>
